File: schematic/bird-cam/bird-cam.kicad_sch (KiCad schematic)
At the start: 28 parts, among them J1 Conn_02x03_Counter_Clockwise, J2 Barrel_Jack, J3 USB_C_Breakout, M1 Stepper_Motor_unipolar_5pin, M2 Stepper_Motor_unipolar_5pin, U1 ATmega328P-P, U2 ESP32-CAM, U3 Stepper_Motor_Driver, U4 Stepper_Motor_Driver, U5 load_cell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

Commit message: bit more schem, still not done
Parts:
- added SW1: SW_SPDT, symbol Switch:SW_SPDT
- added SW2: SW_SPST, symbol Switch:SW_SPST
- added U10: TEL0094, symbol bird-cam:TEL00094
Connections:
- net +5V: now also SW2.2 (B), U10.2 (VCC); no longer C3.1, C4.1, J2.1, J3. (VBUS)
- net ESP32_RX: now also U10.3 (TX)
- net ESP32_TX: now also U10.4 (RX)
- net GND: now also U10.5 (GND)
- net RTC_SCL: now also U1.28 (PC5)
- net RTC_SDA: now also U1.27 (PC4)
- net Vbus: now reaches J3. (VBUS)
- net Vbus: now also C3.1, SW1.1 (A)
- new net: SW1.2 (B), SW2.1 (A)
- new net: U5. (White), U8. (VCC) (x3)
- new net: U6. (White), U7. (VCC) (x3)
- new net GPS_EN: U10.6 (EN)
- new net Vbarrel: C4.1, J2.1, SW1.3 (C)
- no-connect marks 17 -> 18
Other:
- moved on the sheet: C1, C2, U2

Commit message: tentatively finished schem
Parts:
- added NT1, NT2, NT3, NT4: NetTie_2, symbol Device:NetTie_2
Connections:
- net +5V: no longer J1.6 (Pin_6)
- net GPS_EN: now also U2. (VCC)
- net Indicator_LED: now also U1.16 (PB2)
- net Nightlight_LED: now also U1.15 (PB1)
- net Reset: now also J1.6 (Pin_6)
- net load1_DT: now also U1.4 (PD2)
- net load1_SCK: now also U1.5 (PD3)
- net load2_DT: now also U1.11 (PD5)
- net load2_SCK: now also U1.12 (PD6)
- net step1_in1: now also U1.23 (PC0), NT1.1
- net step1_in2: now also U1.24 (PC1), NT2.1
- net step1_in3: now also U1.25 (PC2), NT3.1
- net step1_in4: now also U1.26 (PC3), NT4.1
- net step2_in1: now also NT1.2
- net step2_in2: now also NT2.2
- net step2_in3: now also NT3.2
- net step2_in4: now also NT4.2
- net ESP32_RX2: now reaches U1.3 (PD1)
- net ESP32_RX2: now also U2. (VCC)
- new net: U5. (White), U8. (VCC) (x3)
- new net: U6. (White), U7. (VCC) (x3)
- no-connect marks 18 -> 21
Other:
- moved on the sheet: R1

Commit message: schem edits
Parts:
- U10: now not fitted
Connections:
- net ESP32_RX: now also U1.3 (PD1); no longer U10.3 (TX)
- net ESP32_TX: now also U1.2 (PD0); no longer U10.4 (RX)
- net GPS_EN: no longer U10.6 (EN)
- net Indicator_LED: now also U1.23 (PC0); no longer U1.16 (PB2)
- net step1_in1: now also U1.16 (PB2); no longer U1.23 (PC0)
- removed net ESP32_RX2: U1.3 (PD1), U2. (VCC)
- new net: U5. (White), U8. (VCC) (x3)
- new net: U6. (White), U7. (VCC) (x3)
- no-connect marks 21 -> 25
Changed lines of the file:
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@@
   (no_connect (at 228.6 62.23))
   (no_connect (at 132.08 29.21))
+  (no_connect (at 148.59 31.75))
   (no_connect (at 91.44 113.03))
   (no_connect (at 228.6 105.41))
-  (no_connect (at 228.6 87.63))
   (no_connect (at 101.6 41.91))
+  (no_connect (at 80.01 118.11))
   (no_connect (at 228.6 44.45))
   (no_connect (at 43.18 31.75))
+  (no_connect (at 80.01 125.73))
   (no_connect (at 101.6 36.83))
+  (no_connect (at 80.01 120.65))
   (no_connect (at 198.12 44.45))
   (no_connect (at 48.26 119.38))
@@
   (no_connect (at 101.6 39.37))
   (no_connect (at 228.6 97.79))
+  (no_connect (at 90.17 46.99))
   (no_connect (at 43.18 39.37))
   (wire (pts (xy 223.52 27.94) (xy 223.52 31.75))
@@
     (stroke (width 0) (type default))
   )
-  (wire (pts (xy 241.3 67.31) (xy 228.6 67.31))
+  (wire (pts (xy 243.84 67.31) (xy 228.6 67.31))
     (stroke (width 0) (type default))
   )
@@
     (stroke (width 0) (type default))
   )
+  (wire (pts (xy 228.6 87.63) (xy 241.3 87.63))
+    (stroke (width 0) (type default))
+  )
   (wire (pts (xy 160.02 175.26) (xy 168.91 175.26))
     (stroke (width 0) (type default))
@@
     (stroke (width 0) (type default))
   )
-  (wire (pts (xy 228.6 49.53) (xy 243.84 49.53))
+  (wire (pts (xy 228.6 49.53) (xy 241.3 49.53))
     (stroke (width 0) (type default))
   )
@@
     (effects (font (size 1.27 1.27)) (justify right bottom))
   )
-  (label "ESP32_RX" (at 80.01 118.11 0) (fields_autoplaced)
-    (effects (font (size 1.27 1.27)) (justify left bottom))
-  )
   (label "Osc" (at 236.22 59.69 180) (fields_autoplaced)
     (effects (font (size 1.27 1.27)) (justify right bottom))
@@
     (effects (font (size 1.27 1.27)) (justify right bottom))
   )
-  (label "Indicator_LED" (at 243.84 49.53 180) (fields_autoplaced)
+  (label "Indicator_LED" (at 243.84 67.31 180) (fields_autoplaced)
     (effects (font (size 1.27 1.27)) (justify right bottom))
   )
@@
     (effects (font (size 1.27 1.27)) (justify right bottom))
   )
-  (label "GPS_EN" (at 80.01 125.73 0) (fields_autoplaced)
-    (effects (font (size 1.27 1.27)) (justify left bottom))
-  )
   (label "step1_in3" (at 128.27 144.78 0) (fields_autoplaced)
     (effects (font (size 1.27 1.27)) (justify left bottom))
@@
     (effects (font (size 1.27 1.27)) (justify left bottom))
   )
+  (label "ESP32_RX" (at 241.3 90.17 180) (fields_autoplaced)
+    (effects (font (size 1.27 1.27)) (justify right bottom))
+  )
   (label "coil2_1" (at 194.31 143.51 270) (fields_autoplaced)
     (effects (font (size 1.27 1.27)) (justify right bottom))
@@
     (effects (font (size 1.27 1.27)) (justify right bottom))
   )
-  (label "ESP32_TX" (at 80.01 120.65 0) (fields_autoplaced)
-    (effects (font (size 1.27 1.27)) (justify left bottom))
-  )
   (label "step2_in3" (at 128.27 177.8 0) (fields_autoplaced)
     (effects (font (size 1.27 1.27)) (justify left bottom))
@@
     (effects (font (size 1.27 1.27)) (justify right bottom))
   )
-  (label "ESP32_RX2" (at 148.59 31.75 180) (fields_autoplaced)
-    (effects (font (size 1.27 1.27)) (justify right bottom))
-  )
-  (label "ESP32_RX2" (at 241.3 90.17 180) (fields_autoplaced)
-    (effects (font (size 1.27 1.27)) (justify right bottom))
-  )
   (label "com1" (at 191.77 121.92 270) (fields_autoplaced)
     (effects (font (size 1.27 1.27)) (justify right bottom))
@@
     (effects (font (size 1.27 1.27)) (justify right bottom))
   )
-  (label "step1_in1" (at 241.3 67.31 180) (fields_autoplaced)
+  (label "step1_in1" (at 241.3 49.53 180) (fields_autoplaced)
     (effects (font (size 1.27 1.27)) (justify right bottom))
   )
@@
   )
   (label "step2_in2" (at 163.83 124.46 180) (fields_autoplaced)
+    (effects (font (size 1.27 1.27)) (justify right bottom))
+  )
+  (label "ESP32_TX" (at 241.3 87.63 180) (fields_autoplaced)
     (effects (font (size 1.27 1.27)) (justify right bottom))
   )
@@
   )
   (symbol (lib_id "bird-cam:TEL00094") (at 93.98 128.27 0) (unit 1)
-    (in_bom yes) (on_board yes) (dnp no) (fields_autoplaced)
+    (in_bom yes) (on_board yes) (dnp yes) (fields_autoplaced)
     (property "Reference" "U10" (at 107.315 118.7363 0)
       (effects (font (size 1.27 1.27)) (justify left))

Commit message: everything
Connections:
- net ESP32_R: now reaches U1.6 (PD4)
- net ESP32_R: now also U2. (VCC)
- new net: U5. (White), U8. (VCC) (x3)
- new net: U6. (White), U7. (VCC) (x3)
- no-connect marks 25 -> 24
Changed lines of the file:
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@@
   (junction (at 238.76 133.35) (diameter 0) (color 0 0 0 0)
-  )
-  (junction (at 134.62 46.99) (diameter 0) (color 0 0 0 0)
   )
   (junction (at 257.81 93.98) (diameter 0) (color 0 0 0 0)
@@
   (no_connect (at 132.08 39.37))
   (no_connect (at 101.6 39.37))
-  (no_connect (at 228.6 97.79))
   (no_connect (at 90.17 46.99))
   (no_connect (at 43.18 39.37))
@@
     (stroke (width 0) (type default))
   )
-  (wire (pts (xy 134.62 46.99) (xy 132.08 46.99))
-    (stroke (width 0) (type default))
-  )
   (wire (pts (xy 223.52 24.13) (xy 223.52 27.94))
     (stroke (width 0) (type default))
@@
     (stroke (width 0) (type default))
   )
-  (wire (pts (xy 134.62 49.53) (xy 134.62 46.99))
+  (wire (pts (xy 134.62 36.83) (xy 134.62 49.53))
     (stroke (width 0) (type default))
   )
@@
     (stroke (width 0) (type default))
   )
+  (wire (pts (xy 132.08 46.99) (xy 148.59 46.99))
+    (stroke (width 0) (type default))
+  )
   (wire (pts (xy 160.02 147.32) (xy 168.91 147.32))
     (stroke (width 0) (type default))
@@
     (stroke (width 0) (type default))
   )
+  (wire (pts (xy 228.6 97.79) (xy 241.3 97.79))
+    (stroke (width 0) (type default))
+  )
   (wire (pts (xy 160.02 177.8) (xy 168.91 177.8))
     (stroke (width 0) (type default))
@@
   )
   (wire (pts (xy 121.92 152.4) (xy 139.7 152.4))
-    (stroke (width 0) (type default))
-  )
-  (wire (pts (xy 134.62 36.83) (xy 134.62 46.99))
     (stroke (width 0) (type default))
   )
@@
     (effects (font (size 1.27 1.27)) (justify right bottom))
   )
+  (label "ESP32_R" (at 241.3 97.79 180) (fields_autoplaced)
+    (effects (font (size 1.27 1.27)) (justify right bottom))
+  )
   (label "ESP32_TX" (at 148.59 44.45 180) (fields_autoplaced)
     (effects (font (size 1.27 1.27)) (justify right bottom))
@@
     (effects (font (size 1.27 1.27)) (justify left bottom))
   )
+  (label "ESP32_R" (at 148.59 46.99 180) (fields_autoplaced)
+    (effects (font (size 1.27 1.27)) (justify right bottom))
+  )
   (label "Indicator_LED" (at 278.13 133.35 180) (fields_autoplaced)
